Commit message: switch to gazebo fortress, stop using gazebo classic

File: models/minimal/minimal.xacro (robot description, xacro)
@@ -3,5 +3,5 @@
        xmlns:xacro="http://ros.org/wiki/xacro">
        <xacro:property name="pkg_dir" value="package://rm_sim_bringup"/>
-       <xacro:property name="mesh_file" value="models/minimal/box.stl"/>
+       <xacro:property name="mesh_file" value="models/minimal/box.dae"/>
        <link name="base_link">
     <visual>
