Commit message: switch to gazebo fortress, stop using gazebo classic

File: models/translated_nightbuild/robot_translated.xacro (robot description, xacro)
@@ -16,5 +16,5 @@
       <origin xyz="-0.0186236 0.0777092 0.0547166" rpy="1.5708 -0.122269 0.551744" />
       <geometry>
-        <mesh filename="package://rm_sim_bringup/share/rm_sim_bringup/models/translated_nightbuild/assets/__.stl" />
+        <mesh filename="package://rm_sim_bringup/models/translated_nightbuild/assets/__.stl" />
       </geometry>
       <material name="_material">
@@ -25,5 +25,5 @@
       <origin xyz="-0.0186236 0.0777092 0.0547166" rpy="1.5708 -0.122269 0.551744" />
       <geometry>
-        <mesh filename="package://rm_sim_bringup/share/rm_sim_bringup/models/translated_nightbuild/assets/__.stl" />
+        <mesh filename="package://rm_sim_bringup/models/translated_nightbuild/assets/__.stl" />
       </geometry>
     </collision>
@@ -31,5 +31,5 @@
       <origin xyz="-3.46945e-18 0 0.002" rpy="-1.5708 -0 3.14159" />
       <geometry>
-        <mesh filename="package://rm_sim_bringup/share/rm_sim_bringup/models/translated_nightbuild/assets/ptz_stator_fixed_horizontal.stl" />
+        <mesh filename="package://rm_sim_bringup/models/translated_nightbuild/assets/ptz_stator_fixed_horizontal.stl" />
       </geometry>
       <material name="ptz_stator_fixed_horizontal_material">
@@ -40,5 +40,5 @@
       <origin xyz="-3.46945e-18 0 0.002" rpy="-1.5708 -0 3.14159" />
       <geometry>
-        <mesh filename="package://rm_sim_bringup/share/rm_sim_bringup/models/translated_nightbuild/assets/ptz_stator_fixed_horizontal.stl" />
+        <mesh filename="package://rm_sim_bringup/models/translated_nightbuild/assets/ptz_stator_fixed_horizontal.stl" />
       </geometry>
     </collision>
@@ -46,5 +46,5 @@
       <origin xyz="0.0175 0.184 0.042" rpy="1.5708 1.249e-16 3.14159" />
       <geometry>
-        <mesh filename="package://rm_sim_bringup/share/rm_sim_bringup/models/translated_nightbuild/assets/side_reinforcement_of_collision_bar.stl" />
+        <mesh filename="package://rm_sim_bringup/models/translated_nightbuild/assets/side_reinforcement_of_collision_bar.stl" />
       </geometry>
       <material name="side_reinforcement_of_collision_bar_material">
@@ -55,5 +55,5 @@
       <origin xyz="0.0175 0.184 0.042" rpy="1.5708 1.249e-16 3.14159" />
       <geometry>
-        <mesh filename="package://rm_sim_bringup/share/rm_sim_bringup/models/translated_nightbuild/assets/side_reinforcement_of_collision_bar.stl" />
+        <mesh filename="package://rm_sim_bringup/models/translated_nightbuild/assets/side_reinforcement_of_collision_bar.stl" />
       </geometry>
     </collision>
@@ -61,5 +61,5 @@
       <origin xyz="-0.825677 -0.0211413 0.0745391" rpy="1.5708 5.84832e-16 1.5708" />
       <geometry>
-        <mesh filename="package://rm_sim_bringup/share/rm_sim_bringup/models/translated_nightbuild/assets/anticollision_guide_wheel_fixing_plate.stl" />
+        <mesh filename="package://rm_sim_bringup/models/translated_nightbuild/assets/anticollision_guide_wheel_fixing_plate.stl" />
       </geometry>
       <material name="anticollision_guide_wheel_fixing_plate_material">
@@ -70,5 +70,5 @@
       <origin xyz="-0.825677 -0.0211413 0.0745391" rpy="1.5708 5.84832e-16 1.5708" />
       <geometry>
-        <mesh filename="package://rm_sim_bringup/share/rm_sim_bringup/models/translated_nightbuild/assets/anticollision_guide_wheel_fixing_plate.stl" />
+        <mesh filename="package://rm_sim_bringup/models/translated_nightbuild/assets/anticollision_guide_wheel_fixing_plate.stl" />
       </geometry>
     </collision>
@@ -76,5 +76,5 @@
       <origin xyz="-0.261 0.273 0.042" rpy="-1.5708 2.63678e-16 3.14159" />
       <geometry>
-        <mesh filename="package://rm_sim_bringup/share/rm_sim_bringup/models/translated_nightbuild/assets/front_and_rear_collision_bars.stl" />
+        <mesh filename="package://rm_sim_bringup/models/translated_nightbuild/assets/front_and_rear_collision_bars.stl" />
       </geometry>
       <material name="front_and_rear_collision_bars_material">
@@ -85,5 +85,5 @@
       <origin xyz="-0.261 0.273 0.042" rpy="-1.5708 2.63678e-16 3.14159" />
       <geometry>
-        <mesh filename="package://rm_sim_bringup/share/rm_sim_bringup/models/translated_nightbuild/assets/front_and_rear_collision_bars.stl" />
+        <mesh filename="package://rm_sim_bringup/models/translated_nightbuild/assets/front_and_rear_collision_bars.stl" />
       </geometry>
     </collision>
@@ -91,5 +91,5 @@
       <origin xyz="0.25 0.304 0.022" rpy="1.5708 -6.29205e-16 -1.5708" />
       <geometry>
-        <mesh filename="package://rm_sim_bringup/share/rm_sim_bringup/models/translated_nightbuild/assets/side_impact_bar.stl" />
+        <mesh filename="package://rm_sim_bringup/models/translated_nightbuild/assets/side_impact_bar.stl" />
       </geometry>
       <material name="side_impact_bar_material">
@@ -100,5 +100,5 @@
       <origin xyz="0.25 0.304 0.022" rpy="1.5708 -6.29205e-16 -1.5708" />
       <geometry>
-        <mesh filename="package://rm_sim_bringup/share/rm_sim_bringup/models/translated_nightbuild/assets/side_impact_bar.stl" />
+        <mesh filename="package://rm_sim_bringup/models/translated_nightbuild/assets/side_impact_bar.stl" />
       </geometry>
     </collision>
@@ -106,5 +106,5 @@
       <origin xyz="0.271 0.294 0.0365" rpy="-3.14159 1.94289e-16 3.07755" />
       <geometry>
-        <mesh filename="package://rm_sim_bringup/share/rm_sim_bringup/models/translated_nightbuild/assets/30_6_9guide_wheel.stl" />
+        <mesh filename="package://rm_sim_bringup/models/translated_nightbuild/assets/30_6_9guide_wheel.stl" />
       </geometry>
       <material name="30_6_9guide_wheel_material">
@@ -115,5 +115,5 @@
       <origin xyz="0.271 0.294 0.0365" rpy="-3.14159 1.94289e-16 3.07755" />
       <geometry>
-        <mesh filename="package://rm_sim_bringup/share/rm_sim_bringup/models/translated_nightbuild/assets/30_6_9guide_wheel.stl" />
+        <mesh filename="package://rm_sim_bringup/models/translated_nightbuild/assets/30_6_9guide_wheel.stl" />
       </geometry>
     </collision>
@@ -121,5 +121,5 @@
       <origin xyz="0.0441413 -0.802677 0.0975391" rpy="1.5708 1.249e-16 3.14159" />
       <geometry>
-        <mesh filename="package://rm_sim_bringup/share/rm_sim_bringup/models/translated_nightbuild/assets/anticollision_guide_wheel_fixing_plate.stl" />
+        <mesh filename="package://rm_sim_bringup/models/translated_nightbuild/assets/anticollision_guide_wheel_fixing_plate.stl" />
       </geometry>
       <material name="anticollision_guide_wheel_fixing_plate_2_material">
@@ -130,5 +130,5 @@
       <origin xyz="0.0441413 -0.802677 0.0975391" rpy="1.5708 1.249e-16 3.14159" />
       <geometry>
-        <mesh filename="package://rm_sim_bringup/share/rm_sim_bringup/models/translated_nightbuild/assets/anticollision_guide_wheel_fixing_plate.stl" />
+        <mesh filename="package://rm_sim_bringup/models/translated_nightbuild/assets/anticollision_guide_wheel_fixing_plate.stl" />
       </geometry>
     </collision>
@@ -136,5 +136,5 @@
       <origin xyz="-0.271 0.294 0.0365" rpy="-3.14159 1.94289e-16 3.07755" />
       <geometry>
-        <mesh filename="package://rm_sim_bringup/share/rm_sim_bringup/models/translated_nightbuild/assets/30_6_9guide_wheel.stl" />
+        <mesh filename="package://rm_sim_bringup/models/translated_nightbuild/assets/30_6_9guide_wheel.stl" />
       </geometry>
       <material name="30_6_9guide_wheel_2_material">
@@ -145,5 +145,5 @@
       <origin xyz="-0.271 0.294 0.0365" rpy="-3.14159 1.94289e-16 3.07755" />
       <geometry>
-        <mesh filename="package://rm_sim_bringup/share/rm_sim_bringup/models/translated_nightbuild/assets/30_6_9guide_wheel.stl" />
+        <mesh filename="package://rm_sim_bringup/models/translated_nightbuild/assets/30_6_9guide_wheel.stl" />
       </geometry>
     </collision>
@@ -151,5 +151,5 @@
       <origin xyz="0.261 0.273 0.022" rpy="1.5708 -1.249e-16 -3.05311e-15" />
       <geometry>
-        <mesh filename="package://rm_sim_bringup/share/rm_sim_bringup/models/translated_nightbuild/assets/front_and_rear_collision_bars.stl" />
+        <mesh filename="package://rm_sim_bringup/models/translated_nightbuild/assets/front_and_rear_collision_bars.stl" />
       </geometry>
       <material name="front_and_rear_collision_bars_2_material">
@@ -160,5 +160,5 @@
       <origin xyz="0.261 0.273 0.022" rpy="1.5708 -1.249e-16 -3.05311e-15" />
       <geometry>
-        <mesh filename="package://rm_sim_bringup/share/rm_sim_bringup/models/translated_nightbuild/assets/front_and_rear_collision_bars.stl" />
+        <mesh filename="package://rm_sim_bringup/models/translated_nightbuild/assets/front_and_rear_collision_bars.stl" />
       </geometry>
     </collision>
@@ -166,5 +166,5 @@
       <origin xyz="-0.825677 -0.0211413 0.0975391" rpy="1.5708 5.85187e-16 1.5708" />
       <geometry>
-        <mesh filename="package://rm_sim_bringup/share/rm_sim_bringup/models/translated_nightbuild/assets/anticollision_guide_wheel_fixing_plate.stl" />
+        <mesh filename="package://rm_sim_bringup/models/translated_nightbuild/assets/anticollision_guide_wheel_fixing_plate.stl" />
       </geometry>
       <material name="anticollision_guide_wheel_fixing_plate_3_material">
@@ -175,5 +175,5 @@
       <origin xyz="-0.825677 -0.0211413 0.0975391" rpy="1.5708 5.85187e-16 1.5708" />
       <geometry>
-        <mesh filename="package://rm_sim_bringup/share/rm_sim_bringup/models/translated_nightbuild/assets/anticollision_guide_wheel_fixing_plate.stl" />
+        <mesh filename="package://rm_sim_bringup/models/translated_nightbuild/assets/anticollision_guide_wheel_fixing_plate.stl" />
       </geometry>
     </collision>
@@ -181,5 +181,5 @@
       <origin xyz="0.0441413 -0.802677 0.0745391" rpy="1.5708 1.249e-16 3.14159" />
       <geometry>
-        <mesh filename="package://rm_sim_bringup/share/rm_sim_bringup/models/translated_nightbuild/assets/anticollision_guide_wheel_fixing_plate.stl" />
+        <mesh filename="package://rm_sim_bringup/models/translated_nightbuild/assets/anticollision_guide_wheel_fixing_plate.stl" />
       </geometry>
       <material name="anticollision_guide_wheel_fixing_plate_4_material">
@@ -190,5 +190,5 @@
       <origin xyz="0.0441413 -0.802677 0.0745391" rpy="1.5708 1.249e-16 3.14159" />
       <geometry>
-        <mesh filename="package://rm_sim_bringup/share/rm_sim_bringup/models/translated_nightbuild/assets/anticollision_guide_wheel_fixing_plate.stl" />
+        <mesh filename="package://rm_sim_bringup/models/translated_nightbuild/assets/anticollision_guide_wheel_fixing_plate.stl" />
       </geometry>
     </collision>
@@ -196,5 +196,5 @@
       <origin xyz="1.38778e-17 0.2515 0.046" rpy="1.5708 1.249e-16 3.14159" />
       <geometry>
-        <mesh filename="package://rm_sim_bringup/share/rm_sim_bringup/models/translated_nightbuild/assets/armor_plate_spacer2.stl" />
+        <mesh filename="package://rm_sim_bringup/models/translated_nightbuild/assets/armor_plate_spacer2.stl" />
       </geometry>
       <material name="armor_plate_spacer2_material">
@@ -205,5 +205,5 @@
       <origin xyz="1.38778e-17 0.2515 0.046" rpy="1.5708 1.249e-16 3.14159" />
       <geometry>
-        <mesh filename="package://rm_sim_bringup/share/rm_sim_bringup/models/translated_nightbuild/assets/armor_plate_spacer2.stl" />
+        <mesh filename="package://rm_sim_bringup/models/translated_nightbuild/assets/armor_plate_spacer2.stl" />
       </geometry>
     </collision>
@@ -211,5 +211,5 @@
       <origin xyz="-0.1585 -0.094 0.0395" rpy="1.5708 8.96959e-16 -1.5708" />
       <geometry>
-        <mesh filename="package://rm_sim_bringup/share/rm_sim_bringup/models/translated_nightbuild/assets/side_protective_shell_modified.stl" />
+        <mesh filename="package://rm_sim_bringup/models/translated_nightbuild/assets/side_protective_shell_modified.stl" />
       </geometry>
       <material name="side_protective_shell_modified_material">
@@ -220,5 +220,5 @@
       <origin xyz="-0.1585 -0.094 0.0395" rpy="1.5708 8.96959e-16 -1.5708" />
       <geometry>
-        <mesh filename="package://rm_sim_bringup/share/rm_sim_bringup/models/translated_nightbuild/assets/side_protective_shell_modified.stl" />
+        <mesh filename="package://rm_sim_bringup/models/translated_nightbuild/assets/side_protective_shell_modified.stl" />
       </geometry>
     </collision>
@@ -226,5 +226,5 @@
       <origin xyz="0.14 -0.083 0.003" rpy="1.5708 1.47105e-15 3.14159" />
       <geometry>
-        <mesh filename="package://rm_sim_bringup/share/rm_sim_bringup/models/translated_nightbuild/assets/stringer_port.stl" />
+        <mesh filename="package://rm_sim_bringup/models/translated_nightbuild/assets/stringer_port.stl" />
       </geometry>
       <material name="stringer_port_material">
@@ -235,5 +235,5 @@
       <origin xyz="0.14 -0.083 0.003" rpy="1.5708 1.47105e-15 3.14159" />
       <geometry>
-        <mesh filename="package://rm_sim_bringup/share/rm_sim_bringup/models/translated_nightbuild/assets/stringer_port.stl" />
+        <mesh filename="package://rm_sim_bringup/models/translated_nightbuild/assets/stringer_port.stl" />
       </geometry>
     </collision>
@@ -241,5 +241,5 @@
       <origin xyz="0.14 0.083 0.003" rpy="1.5708 4.02456e-16 -3.14159" />
       <geometry>
-        <mesh filename="package://rm_sim_bringup/share/rm_sim_bringup/models/translated_nightbuild/assets/sill_reinforcing.stl" />
+        <mesh filename="package://rm_sim_bringup/models/translated_nightbuild/assets/sill_reinforcing.stl" />
       </geometry>
       <material name="sill_reinforcing_material">
@@ -250,5 +250,5 @@
       <origin xyz="0.14 0.083 0.003" rpy="1.5708 4.02456e-16 -3.14159" />
       <geometry>
-        <mesh filename="package://rm_sim_bringup/share/rm_sim_bringup/models/translated_nightbuild/assets/sill_reinforcing.stl" />
+        <mesh filename="package://rm_sim_bringup/models/translated_nightbuild/assets/sill_reinforcing.stl" />
       </geometry>
     </collision>
@@ -256,5 +256,5 @@
       <origin xyz="-0.1485 -0.093 0.0385" rpy="1.5708 -8.73324e-17 -1.5708" />
       <geometry>
-        <mesh filename="package://rm_sim_bringup/share/rm_sim_bringup/models/translated_nightbuild/assets/side_protective_shell02.stl" />
+        <mesh filename="package://rm_sim_bringup/models/translated_nightbuild/assets/side_protective_shell02.stl" />
       </geometry>
       <material name="side_protective_shell02_material">
@@ -265,5 +265,5 @@
       <origin xyz="-0.1485 -0.093 0.0385" rpy="1.5708 -8.73324e-17 -1.5708" />
       <geometry>
-        <mesh filename="package://rm_sim_bringup/share/rm_sim_bringup/models/translated_nightbuild/assets/side_protective_shell02.stl" />
+        <mesh filename="package://rm_sim_bringup/models/translated_nightbuild/assets/side_protective_shell02.stl" />
       </geometry>
     </collision>
@@ -271,5 +271,5 @@
       <origin xyz="-0.1805 -0.09 0.129" rpy="1.5708 6.42557e-16 1.5708" />
       <geometry>
-        <mesh filename="package://rm_sim_bringup/share/rm_sim_bringup/models/translated_nightbuild/assets/sca_m3_l10_ver1.stl" />
+        <mesh filename="package://rm_sim_bringup/models/translated_nightbuild/assets/sca_m3_l10_ver1.stl" />
       </geometry>
       <material name="sca_m3_l10_ver1_material">
@@ -280,5 +280,5 @@
       <origin xyz="-0.1805 -0.09 0.129" rpy="1.5708 6.42557e-16 1.5708" />
       <geometry>
-        <mesh filename="package://rm_sim_bringup/share/rm_sim_bringup/models/translated_nightbuild/assets/sca_m3_l10_ver1.stl" />
+        <mesh filename="package://rm_sim_bringup/models/translated_nightbuild/assets/sca_m3_l10_ver1.stl" />
       </geometry>
     </collision>
@@ -286,5 +286,5 @@
       <origin xyz="-0.2145 -2.77556e-16 0.046" rpy="1.5708 6.42557e-16 1.5708" />
       <geometry>
-        <mesh filename="package://rm_sim_bringup/share/rm_sim_bringup/models/translated_nightbuild/assets/armor_plate_spacer.stl" />
+        <mesh filename="package://rm_sim_bringup/models/translated_nightbuild/assets/armor_plate_spacer.stl" />
       </geometry>
       <material name="armor_plate_spacer_material">
@@ -295,5 +295,5 @@
       <origin xyz="-0.2145 -2.77556e-16 0.046" rpy="1.5708 6.42557e-16 1.5708" />
       <geometry>
-        <mesh filename="package://rm_sim_bringup/share/rm_sim_bringup/models/translated_nightbuild/assets/armor_plate_spacer.stl" />
+        <mesh filename="package://rm_sim_bringup/models/translated_nightbuild/assets/armor_plate_spacer.stl" />
       </geometry>
     </collision>
@@ -301,5 +301,5 @@
       <origin xyz="0.223069 -0.094 0.0915261" rpy="1.309 -4.44684e-16 1.5708" />
       <geometry>
-        <mesh filename="package://rm_sim_bringup/share/rm_sim_bringup/models/translated_nightbuild/assets/front_and_rear_protective_covers.stl" />
+        <mesh filename="package://rm_sim_bringup/models/translated_nightbuild/assets/front_and_rear_protective_covers.stl" />
       </geometry>
       <material name="front_and_rear_protective_covers_material">
@@ -310,5 +310,5 @@
       <origin xyz="0.223069 -0.094 0.0915261" rpy="1.309 -4.44684e-16 1.5708" />
       <geometry>
-        <mesh filename="package://rm_sim_bringup/share/rm_sim_bringup/models/translated_nightbuild/assets/front_and_rear_protective_covers.stl" />
+        <mesh filename="package://rm_sim_bringup/models/translated_nightbuild/assets/front_and_rear_protective_covers.stl" />
       </geometry>
     </collision>
@@ -316,5 +316,5 @@
       <origin xyz="0.196 -0.077 -0.001" rpy="3.14159 1.52656e-15 3.14159" />
       <geometry>
-        <mesh filename="package://rm_sim_bringup/share/rm_sim_bringup/models/translated_nightbuild/assets/rfidmount.stl" />
+        <mesh filename="package://rm_sim_bringup/models/translated_nightbuild/assets/rfidmount.stl" />
       </geometry>
       <material name="rfidmount_material">
@@ -325,5 +325,5 @@
       <origin xyz="0.196 -0.077 -0.001" rpy="3.14159 1.52656e-15 3.14159" />
       <geometry>
-        <mesh filename="package://rm_sim_bringup/share/rm_sim_bringup/models/translated_nightbuild/assets/rfidmount.stl" />
+        <mesh filename="package://rm_sim_bringup/models/translated_nightbuild/assets/rfidmount.stl" />
       </geometry>
     </collision>
@@ -331,5 +331,5 @@
       <origin xyz="0.259 -0.1265 -0.022" rpy="1.5708 6.42557e-16 1.5708" />
       <geometry>
-        <mesh filename="package://rm_sim_bringup/share/rm_sim_bringup/models/translated_nightbuild/assets/flying_ramp_guide_wheel_connecting_plate.stl" />
+        <mesh filename="package://rm_sim_bringup/models/translated_nightbuild/assets/flying_ramp_guide_wheel_connecting_plate.stl" />
       </geometry>
       <material name="flying_ramp_guide_wheel_connecting_plate_material">
@@ -340,5 +340,5 @@
       <origin xyz="0.259 -0.1265 -0.022" rpy="1.5708 6.42557e-16 1.5708" />
       <geometry>
-        <mesh filename="package://rm_sim_bringup/share/rm_sim_bringup/models/translated_nightbuild/assets/flying_ramp_guide_wheel_connecting_plate.stl" />
+        <mesh filename="package://rm_sim_bringup/models/translated_nightbuild/assets/flying_ramp_guide_wheel_connecting_plate.stl" />
       </geometry>
     </collision>
@@ -346,5 +346,5 @@
       <origin xyz="-0.1855 0.09 0.13" rpy="1.5708 -7.43849e-15 4.18358e-15" />
       <geometry>
-        <mesh filename="package://rm_sim_bringup/share/rm_sim_bringup/models/translated_nightbuild/assets/flying_ramp_guide_wheel_adapter.stl" />
+        <mesh filename="package://rm_sim_bringup/models/translated_nightbuild/assets/flying_ramp_guide_wheel_adapter.stl" />
       </geometry>
       <material name="flying_ramp_guide_wheel_adapter_material">
@@ -355,5 +355,5 @@
       <origin xyz="-0.1855 0.09 0.13" rpy="1.5708 -7.43849e-15 4.18358e-15" />
       <geometry>
-        <mesh filename="package://rm_sim_bringup/share/rm_sim_bringup/models/translated_nightbuild/assets/flying_ramp_guide_wheel_adapter.stl" />
+        <mesh filename="package://rm_sim_bringup/models/translated_nightbuild/assets/flying_ramp_guide_wheel_adapter.stl" />
       </geometry>
     </collision>
@@ -361,5 +361,5 @@
       <origin xyz="-0.21 -0.1185 0.034" rpy="1.5708 8.32667e-17 -5.20417e-16" />
       <geometry>
-        <mesh filename="package://rm_sim_bringup/share/rm_sim_bringup/models/translated_nightbuild/assets/flying_ramp_guide_wheel_adapter.stl" />
+        <mesh filename="package://rm_sim_bringup/models/translated_nightbuild/assets/flying_ramp_guide_wheel_adapter.stl" />
       </geometry>
       <material name="flying_ramp_guide_wheel_adapter_2_material">
@@ -370,5 +370,5 @@
       <origin xyz="-0.21 -0.1185 0.034" rpy="1.5708 8.32667e-17 -5.20417e-16" />
       <geometry>
-        <mesh filename="package://rm_sim_bringup/share/rm_sim_bringup/models/translated_nightbuild/assets/flying_ramp_guide_wheel_adapter.stl" />
+        <mesh filename="package://rm_sim_bringup/models/translated_nightbuild/assets/flying_ramp_guide_wheel_adapter.stl" />
       </geometry>
     </collision>
@@ -376,5 +376,5 @@
       <origin xyz="-0.1605 0.083 0.022" rpy="1.5708 -4.02456e-16 1.62259e-15" />
       <geometry>
-        <mesh filename="package://rm_sim_bringup/share/rm_sim_bringup/models/translated_nightbuild/assets/middle_longitudinal_beam.stl" />
+        <mesh filename="package://rm_sim_bringup/models/translated_nightbuild/assets/middle_longitudinal_beam.stl" />
       </geometry>
       <material name="middle_longitudinal_beam_material">
@@ -385,5 +385,5 @@
       <origin xyz="-0.1605 0.083 0.022" rpy="1.5708 -4.02456e-16 1.62259e-15" />
       <geometry>
-        <mesh filename="package://rm_sim_bringup/share/rm_sim_bringup/models/translated_nightbuild/assets/middle_longitudinal_beam.stl" />
+        <mesh filename="package://rm_sim_bringup/models/translated_nightbuild/assets/middle_longitudinal_beam.stl" />
       </geometry>
     </collision>
@@ -391,5 +391,5 @@
       <origin xyz="0.255 0.082 -0.008" rpy="-2.54477e-15 1.58207e-15 3.14159" />
       <geometry>
-        <mesh filename="package://rm_sim_bringup/share/rm_sim_bringup/models/translated_nightbuild/assets/lower_protective_plate.stl" />
+        <mesh filename="package://rm_sim_bringup/models/translated_nightbuild/assets/lower_protective_plate.stl" />
       </geometry>
       <material name="lower_protective_plate_material">
@@ -400,5 +400,5 @@
       <origin xyz="0.255 0.082 -0.008" rpy="-2.54477e-15 1.58207e-15 3.14159" />
       <geometry>
-        <mesh filename="package://rm_sim_bringup/share/rm_sim_bringup/models/translated_nightbuild/assets/lower_protective_plate.stl" />
+        <mesh filename="package://rm_sim_bringup/models/translated_nightbuild/assets/lower_protective_plate.stl" />
       </geometry>
     </collision>
@@ -406,5 +406,5 @@
       <origin xyz="-0.13 0.093 0.042" rpy="1.5708 -5.45259e-17 -1.5708" />
       <geometry>
-        <mesh filename="package://rm_sim_bringup/share/rm_sim_bringup/models/translated_nightbuild/assets/front_mounting_plate_modified.stl" />
+        <mesh filename="package://rm_sim_bringup/models/translated_nightbuild/assets/front_mounting_plate_modified.stl" />
       </geometry>
       <material name="front_mounting_plate_modified_material">
@@ -415,5 +415,5 @@
       <origin xyz="-0.13 0.093 0.042" rpy="1.5708 -5.45259e-17 -1.5708" />
       <geometry>
-        <mesh filename="package://rm_sim_bringup/share/rm_sim_bringup/models/translated_nightbuild/assets/front_mounting_plate_modified.stl" />
+        <mesh filename="package://rm_sim_bringup/models/translated_nightbuild/assets/front_mounting_plate_modified.stl" />
       </geometry>
     </collision>
@@ -421,5 +421,5 @@
       <origin xyz="0.259 0.1225 -0.022" rpy="1.5708 6.42557e-16 1.5708" />
       <geometry>
-        <mesh filename="package://rm_sim_bringup/share/rm_sim_bringup/models/translated_nightbuild/assets/flying_ramp_guide_wheel_connecting_plate.stl" />
+        <mesh filename="package://rm_sim_bringup/models/translated_nightbuild/assets/flying_ramp_guide_wheel_connecting_plate.stl" />
       </geometry>
       <material name="flying_ramp_guide_wheel_connecting_plate_2_material">
@@ -430,5 +430,5 @@
       <origin xyz="0.259 0.1225 -0.022" rpy="1.5708 6.42557e-16 1.5708" />
       <geometry>
-        <mesh filename="package://rm_sim_bringup/share/rm_sim_bringup/models/translated_nightbuild/assets/flying_ramp_guide_wheel_connecting_plate.stl" />
+        <mesh filename="package://rm_sim_bringup/models/translated_nightbuild/assets/flying_ramp_guide_wheel_connecting_plate.stl" />
       </geometry>
     </collision>
@@ -436,5 +436,5 @@
       <origin xyz="-0.14 -4.30211e-16 -0.001" rpy="1.5708 3.88578e-16 1.11022e-16" />
       <geometry>
-        <mesh filename="package://rm_sim_bringup/share/rm_sim_bringup/models/translated_nightbuild/assets/armor_plate_protective_plate02.stl" />
+        <mesh filename="package://rm_sim_bringup/models/translated_nightbuild/assets/armor_plate_protective_plate02.stl" />
       </geometry>
       <material name="armor_plate_protective_plate02_material">
@@ -445,5 +445,5 @@
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